File: AlTherm_PCB/AlTherm_PCB.kicad_pcb (KiCad board)
At the start: 2 copper layers, 60 x 100 mm, 59 parts, among them J1 Conn_charger, J2 Conn_Batt, J3 Conn_buzzer, J4 ISP1, J5 Conn_I2C_spare, J6 Conn_SPI_spare, J7 Conn_TempSensor, J8 Conn_LCD, Q1 DMP1045U, SW1 Power Switch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

Commit message: PCB final?
Parts:
- removed J3: Conn_buzzer, Connector_PinHeader_2.54mm:PinHeader_1x02_P2.54mm_Vertical
- removed J6: Conn_SPI_spare, Connector_PinHeader_2.54mm:PinHeader_1x06_P2.54mm_Vertical
- added BZ1: Buzzer, AlarmThermometer:SMA21_pin, F.Cu at (135.5, 53.0)
- added C19: 10uF, Capacitor_SMD:C_1206_3216Metric, F.Cu at (132.5, 40.0)
- added C20: 1.5nF, Capacitor_SMD:C_1206_3216Metric, F.Cu at (155.5, 43.5)
- added C21: 33uF, Capacitor_SMD:C_1206_3216Metric, F.Cu at (122.0, 53.0)
- added L1: 22uH, AlarmThermometer:RS_Type16_Inductor, F.Cu at (124.0, 41.5)
- added R13: 10k, Resistor_SMD:R_1206_3216Metric, F.Cu at (130.0, 110.8)
- added R17: 10k, Resistor_SMD:R_1206_3216Metric, F.Cu at (122.2, 115.5)
- added R18: 10k, Resistor_SMD:R_1206_3216Metric, F.Cu at (148.5, 100.2)
- added R19: 10k, Resistor_SMD:R_1206_3216Metric, F.Cu at (129.5, 92.8)
- added R20: 10k, Resistor_SMD:R_1206_3216Metric, F.Cu at (136.1, 95.2)
- added R21: 10k, Resistor_SMD:R_1206_3216Metric, F.Cu at (136.5, 110.8)
- added R22: 10k, Resistor_SMD:R_1206_3216Metric, F.Cu at (143.5, 110.8)
- added R23: 10K, Resistor_SMD:R_1206_3216Metric, F.Cu at (155.5, 51.5)
- added R24: 560, Resistor_SMD:R_1206_3216Metric, F.Cu at (155.5, 47.5)
- added U8: NCP1403, Package_SO:TSOP-5_1.65x3.05mm_P0.95mm, F.Cu at (122.5, 48.0)
- C15: value 1uF -> 0.1uF
- D3: value LED_active -> Diode_B130-E3; footprint LED_SMD:LED_0805_2012Metric -> Diode_SMD:D_SOD-123
- J2: footprint Connector_PinSocket_2.54mm:PinSocket_1x02_P2.54mm_Vertical -> Connector_PinHeader_2.54mm:PinHeader_1x02_P2.54mm_Vertical
- J5: value Conn_I2C_spare -> Conn_AUX; footprint Connector_PinHeader_2.54mm:PinHeader_1x04_P2.54mm_Vertical -> Connector_PinHeader_2.54mm:PinHeader_1x05_P2.54mm_Vertical
- R15: value 220 -> R_Small
- R16: value 1K -> 10k
- R5, R6, R7, R8: value 10k -> 5k
- SW1: footprint AlarmThermometer:switch_tactile_4pin -> AlarmThermometer:SW_OnOff_12mm
- SW3, SW4, SW5, SW6: footprint AlarmThermometer:switch_tactile_4pin -> AlarmThermometer:SW_MOM_12mm
- U7: value MMA8653FCR1 -> SN54HC14; footprint Package_DFN_QFN:DFN-10_2x2mm_P0.4mm -> AlarmThermometer:SOIC-14W_4x8.75mm_P1.27mm
- moved C5 87.8 mm to (116.0, 57.8), turned to 180 degrees
- moved R1 86.9 mm to (122.0, 57.8)
- moved C8 83.2 mm to (110.0, 57.8)
- moved C11 81.3 mm to (155.5, 55.5)
- moved U4 80.9 mm to (117.5, 63.2)
- moved R15 52.3 mm to (139.0, 40.0), turned to 0 degrees
- moved C18 45.6 mm to (148.5, 53.5), turned to 270 degrees
- moved J2 45.1 mm to (168.0, 125.8), turned to 180 degrees
- moved D3 44.2 mm to (148.5, 47.0), turned to 270 degrees
- moved R12 40.0 mm to (150.8, 80.2), turned to 180 degrees
- moved C4 39.7 mm to (124.5, 62.5), turned to 180 degrees
- moved U5 39.4 mm to (123.0, 90.0), turned to 90 degrees
- moved C17 37.2 mm to (148.5, 60.0), turned to 270 degrees
- moved R11 35.1 mm to (150.8, 85.0)
- moved J4 34.6 mm to (157.8, 85.0)
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Connections:
- C13 pad 1: Net-(C13-Pad1) -> /MNU_IN
- C14 pad 1: VCC -> /UP_IN
- C15 pad 1: VCC -> /DWN_IN
- C16 pad 1: VCC -> /SEL_IN
- D3 pad 1: GND -> Net-(BZ1-Pad1)
- J7 pad 3: /INTO -> /INTI
- R14 pad 1: /INTO -> /INTI
- R15 pad 1: Net-(D3-Pad2) -> /BZR
- R15 pad 2: Net-(R15-Pad2) -> GND
- R16 pad 1: Net-(R16-Pad1) -> VCC
- R16 pad 2: GND -> Net-(R16-Pad2)
- R7 pad 2: /SDL -> /SCL
- SW3 pad 1: /MNU -> GND
- SW3 pad 2: GND -> Net-(R13-Pad2)
- SW4 pad 1: /UP -> GND
- SW4 pad 2: GND -> Net-(R16-Pad2)
- SW5 pad 1: /DWN -> GND
- SW5 pad 2: GND -> Net-(R17-Pad2)
- SW6 pad 1: /SEL -> GND
- SW6 pad 2: GND -> Net-(R18-Pad2)
- U2 pad 11: /SDL -> /SCL
- U2 pad 8: Net-(U2-Pad8) -> (no net)
- U6 pad 1: Net-(U6-Pad1) -> /RESET
- U6 pad 2: Net-(U6-Pad2) -> (no net)
- U6 pad 23: /MNU -> /UP
- U6 pad 24: /SS -> (no net)
- U6 pad 25: Net-(R15-Pad2) -> (no net)
- U6 pad 26: Net-(U6-Pad26) -> (no net)
- U6 pad 6: /UP -> /MNU
- U7 pad 1: VCC -> /UP_IN
- U7 pad 10: /SDA -> (no net)
- U7 pad 2: /SCL -> /UP
- U7 pad 3: /INTI -> /MNU_IN
- U7 pad 4: Net-(C13-Pad1) -> /MNU
- U7 pad 5: Net-(R16-Pad1) -> /DWN_IN
- U7 pad 6: GND -> /DWN
- U7 pad 8: VCC -> /SEL
- U7 pad 9: GND -> /SEL_IN
Routing:
- net GND: track 0.00 -> 451.4 mm, vias 0 -> 7
- net VCC: track 0.00 -> 274.9 mm
- net /SDA: track 0.00 -> 168.5 mm, vias 0 -> 1
- net /SCL: track 0.00 -> 151.7 mm, vias 0 -> 2
- net Net-(C9-Pad1): track 0.00 -> 112.1 mm, vias 0 -> 2
- net Net-(C6-Pad1): track 0.00 -> 97.3 mm, vias 0 -> 1
- net /BZR: track 0.00 -> 82.5 mm
- net Net-(C3-Pad1): track 0.00 -> 79.7 mm
- net Net-(D1-Pad1): track 0.00 -> 70.0 mm, vias 0 -> 2
- net /MNU: track 0.00 -> 69.0 mm
- net /UP: track 0.00 -> 64.6 mm
- net /MOSI: track 0.00 -> 56.8 mm
- net /RESET: track 0.00 -> 56.5 mm
- net Net-(C1-Pad1): track 0.00 -> 53.6 mm
- net Net-(C20-Pad2): track 0.00 -> 53.3 mm
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- added copper zone on B.Cu, net GND
- added copper zone on F.Cu, net GND
Other:
- board size 60 x 100 mm -> 72 x 100 mm
- rule pad_to_mask_clearance: 0.051 -> 0
- board text added: "AUX I2C"
- board text added: "BATT"
- board text added: "CHARGE"
- board text added: "ISP"
- board text added: "RTC"
- board text added: "TEMP"
- board text added: "The Stopford "Alarm-O-Matic" Alarm Thermometer"
- board text added: "VERSION 1.2"
